File: 4ch_mosfet_switch.brd (EAGLE design)
At the start: 49.5 x 49.5 mm, 19 parts, among them Q1 N-CH, Q2 N-CH, Q3 N-CH, Q4 N-CH, X1 CH2, X2 CH1, X3 CH3, X4 CH4

Commit message: Updated Names
Other:
- board text added: "Scott Gibson"
Changed lines of the file:
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@@
 <text x="8.89" y="21.59" size="1.27" layer="27">4ch_mosfet_switch</text>
 <text x="8.89" y="19.05" size="1.27" layer="27">V1.0</text>
+<text x="53.34" y="-10.16" size="1.778" layer="21">Scott Gibson</text>
 </plain>
 <attributes>
