File: 4ch_mosfet_switch.sch (EAGLE design)
At the start: 19 parts, among them Q1 N-CH, Q2 N-CH, Q3 N-CH, Q4 N-CH, X1 CH2, X2 CH1, X3 CH3, X4 CH4

Commit message: Updated Names
Other:
- note added: "Scott Gibson"
Changed lines of the file:
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@@
 <sheet>
 <plain>
+<text x="152.4" y="2.54" size="2.54" layer="94">Scott Gibson</text>
 </plain>
 <instances>
